File: electronics/power/power.kicad_pcb (KiCad board)
At the start: 2 copper layers, 10 parts, among them CON1 5V, J1 RJ45, J2 RJ45, J3 USB_A, P1 CONN_02X05

Commit message: plot boards
Connections:
- J1 pad Hole: (no net) -> GND
- J2 pad : (no net) -> GND
Changed lines of the file:
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@@
 (kicad_pcb (version 4) (host pcbnew "(2015-11-08 BZR 6303, Git 5897580)-product")
   (general
-    (links 32)
+    (links 36)
     (no_connects 5)
-    (area 0 0 0 0)
+    (area 104.460714 65.5495 167.001786 120.40376)
     (thickness 1.6)
     (drawings 0)
@@
     (mod_text_size 1 1)
     (mod_text_width 0.15)
-    (pad_size 2.99974 2.99974)
-    (pad_drill 2.99974)
+    (pad_size 3.64998 3.64998)
+    (pad_drill 3.2512)
     (pad_to_mask_clearance 0.2)
     (aux_axis_origin 0 0)
     (visible_elements FFFFF71F)
     (pcbplotparams
-      (layerselection 0x00030_80000001)
+      (layerselection 0x00000_80000000)
       (usegerberextensions false)
       (excludeedgelayer true)
@@
       (padsonsilk false)
       (subtractmaskfromsilk false)
-      (outputformat 1)
+      (outputformat 5)
       (mirror false)
       (drillshape 1)
@@
     (pad 8 thru_hole oval (at 4.445 -8.89 90) (size 1.8 2.3) (drill 0.89916) (layers *.Cu *.Mask F.SilkS)
       (net 2 "Net-(J1-Pad1)"))
-    (pad "" np_thru_hole oval (at -3.4925 0.9525 90) (size 3 3) (drill 3) (layers *.Cu *.Mask F.SilkS))
-    (pad "" np_thru_hole oval (at 3.4925 0.9525 90) (size 3 3) (drill 3) (layers *.Cu *.Mask F.SilkS))
+    (pad "" thru_hole oval (at -3.4925 0.9525 90) (size 3 3) (drill 3) (layers *.Cu *.Mask F.SilkS)
+      (net 1 GND) (zone_connect 2))
+    (pad "" thru_hole oval (at 3.4925 0.9525 90) (size 3 3) (drill 3) (layers *.Cu *.Mask F.SilkS)
+      (net 1 GND) (zone_connect 2))
     (model Connect/RJ45_8.wrl
       (at (xyz 0 0 0))
@@
     (fp_line (start -7.62 10.7315) (end 7.62 10.7315) (layer F.SilkS) (width 0.15))
     (fp_line (start 7.62 -10.16) (end -7.62 -10.16) (layer F.SilkS) (width 0.15))
-    (pad Hole np_thru_hole circle (at 5.93852 0 270) (size 3.64998 3.64998) (drill 3.2512) (layers *.Cu *.SilkS *.Mask))
-    (pad Hole np_thru_hole circle (at -5.9309 0 270) (size 3.64998 3.64998) (drill 3.2512) (layers *.Cu *.SilkS *.Mask))
+    (pad Hole thru_hole circle (at 5.93852 0 270) (size 3.64998 3.64998) (drill 3.2512) (layers *.Cu *.Mask F.SilkS)
+      (net 1 GND) (zone_connect 2))
+    (pad Hole thru_hole circle (at -5.9309 0 270) (size 3.64998 3.64998) (drill 3.2512) (layers *.Cu *.Mask F.SilkS)
+      (net 1 GND) (zone_connect 2))
     (pad 1 thru_hole rect (at -4.445 -6.35 270) (size 1.8 2.3) (drill 0.89916) (layers *.Cu *.Mask F.SilkS)
       (net 2 "Net-(J1-Pad1)"))
